File: kicad/polkupyörän-takavalo.kicad_pcb (KiCad board)
At the start: 2 copper layers, 40 x 40 mm, 15 parts, among them J1 Conn_01x06_Pin, SW1 SW_Push, U1 STM32G030F6Px

Commit message: version 2
Parts:
- added J2: Conn_ARM_JTAG_SWD_10, Connector_PinHeader_1.27mm:PinHeader_2x05_P1.27mm_Vertical_SMD, F.Cu at (178.1, 110.0)
Connections:
- U1 pad 18: unconnected-(U1-PA13-Pad18) -> Net-(J2-SWDIO/TMS)
- U1 pad 19: unconnected-(U1-PA14/PA15-Pad19) -> Net-(J2-SWCLK/TCK)
Routing:
- net Net-(J2-~{RESET}): track 69.7 -> 122.5 mm
- net VCC: track 67.1 -> 90.4 mm
- net Net-(J2-SWCLK/TCK): track 0.00 -> 20.2 mm, vias 0 -> 2
- net Net-(J2-SWDIO/TMS): track 0.00 -> 19.7 mm, vias 0 -> 2
Other:
- board text added: "rev 0.2 Minix Design"
