File: kicad/polkupyörän-takavalo.kicad_sch (KiCad schematic)
At the start: 15 parts, among them J1 Conn_01x06_Pin, SW1 SW_Push, U1 STM32G030F6Px

Commit message: version 2
Parts:
- added J2: Conn_ARM_JTAG_SWD_10, Connector_PinHeader_1.27mm:PinHeader_2x05_P1.27mm_Vertical_SMD, symbol Connector:Conn_ARM_JTAG_SWD_10
- D1: LCSC C72038 -> C2286
Connections:
- net GND: now also J2.3 (GND), J2.5 (GND), J2.9 (GNDDetect)
- net VCC: now also J2.1 (VTref)
- net at C1.1, R2.2, SW1.2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: now also J2.10 (~{RESET})
- net at U1.18 (PA13): now also J2.2 (SWDIO/TMS)
- net at U1.19 (PA14/PA15): now also J2.4 (SWCLK/TCK)
